File: TSOL_102A.sch (EAGLE design)
At the start: 13 parts, among them X1 BU-SMA-G, X2 BU-SMA-G

Commit message: sch brd updated
Parts:
- removed X2: BU-SMA-G, con-coax:BU-SMA-G
Connections:
- removed net N$1: U$1.RF1, X2.1
Changed lines of the file:
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@@
 <setting verticaltext="up"/>
 </settings>
-<grid distance="0.1" unitdist="inch" unit="inch" style="lines" multiple="1" display="yes" altdistance="0.01" altunitdist="inch" altunit="inch"/>
+<grid distance="0.1" unitdist="inch" unit="inch" style="lines" multiple="1" display="no" altdistance="0.01" altunitdist="inch" altunit="inch"/>
 <layers>
 <layer number="1" name="Top" color="4" fill="1" visible="no" active="no"/>
@@
 <part name="GND4" library="supply1" library_urn="urn:adsk.eagle:library:371" deviceset="GND" device=""/>
 <part name="X1" library="con-coax" library_urn="urn:adsk.eagle:library:133" deviceset="BU-SMA-G" device="" package3d_urn="urn:adsk.eagle:package:6205/1"/>
-<part name="X2" library="con-coax" library_urn="urn:adsk.eagle:library:133" deviceset="BU-SMA-G" device="" package3d_urn="urn:adsk.eagle:package:6205/1"/>
 <part name="GND5" library="SparkFun-PowerSymbols" deviceset="GND" device=""/>
 <part name="GND6" library="SparkFun-PowerSymbols" deviceset="GND" device=""/>
@@
 <instance part="GND4" gate="1" x="68.58" y="-17.78"/>
 <instance part="X1" gate="G1" x="124.46" y="78.74" rot="MR0"/>
-<instance part="X2" gate="G1" x="-15.24" y="60.96"/>
 <instance part="GND5" gate="1" x="121.92" y="68.58"/>
 <instance part="GND6" gate="1" x="93.98" y="10.16"/>
@@
 </segment>
 </net>
-<net name="N$1" class="0">
-<segment>
-<pinref part="X2" gate="G1" pin="1"/>
-<pinref part="U$1" gate="G$1" pin="RF1"/>
-<wire x1="-12.7" y1="60.96" x2="22.86" y2="60.96" width="0.1524" layer="91"/>
-</segment>
-</net>
